Commit message: start nav2 and SLAM

File: src/description/robot_core.xacro (robot description, xacro)
@@ -19,4 +19,12 @@
     <!-- Base Link -->
     <link name="base_link"/>
+    <!-- Base Footprint Link-->
+    <joint name="base_footprint_joint" type="fixed">
+        <parent link="base_link"/>
+        <child link="base_footprint"/>
+        <origin xyz="0 0 0" rpy="0 0 0"/>
+    </joint>
+    <link name="base_footprint">
+    </link>
     <!-- Chassis Link -->
     <joint name="chassis_joint" type="fixed">

Commit message: Revert "start nav2 and SLAM"
This reverts commit e5f2c0530f69068f3d4e7569b421fb95baead006.

File: src/description/robot_core.xacro (robot description, xacro)
@@ -19,12 +19,4 @@
     <!-- Base Link -->
     <link name="base_link"/>
-    <!-- Base Footprint Link-->
-    <joint name="base_footprint_joint" type="fixed">
-        <parent link="base_link"/>
-        <child link="base_footprint"/>
-        <origin xyz="0 0 0" rpy="0 0 0"/>
-    </joint>
-    <link name="base_footprint">
-    </link>
     <!-- Chassis Link -->
     <joint name="chassis_joint" type="fixed">

Commit message: Add initial SLAM

File: src/description/robot_core.xacro (robot description, xacro)
@@ -19,4 +19,11 @@
     <!-- Base Link -->
     <link name="base_link"/>
+    <!-- Base Footprint Link -->
+    <joint name="base_footprint_joint" type="fixed">
+        <parent link="base_link"/>
+        <child link="base_footprint"/>
+        <origin xyz="0 0 0" rpy="0 0 0"/>
+    </joint>
+    <link name="base_footprint"/>
     <!-- Chassis Link -->
     <joint name="chassis_joint" type="fixed">
