Commit message: Get ros2_control working
Note: Kind of finnicky and odom frame is wrong

File: src/description/gazebo_control.xacro (robot description, xacro)
@@ -24,4 +24,9 @@
             <joint_name>DS_Joint</joint_name>
             <joint_name>PS_Joint</joint_name>
+            <joint_name>DW_Joint</joint_name>
+            <joint_name>PW_Joint</joint_name>
+            <joint_name>LoaderJoint</joint_name>
+            <joint_name>HopperJoint</joint_name>
+            <joint_name>DoorJoint</joint_name>
         </plugin>
     </gazebo>

File: src/description/ros2_control.xacro (robot description, xacro)
@@ -29,4 +29,21 @@
                 <state_interface name="position"/>
             </joint>
+            <joint name="DW_Joint">
+                <state_interface name="position"/>
+                <state_interface name="velocity"/>
+            </joint>
+            <joint name="PW_Joint">
+                <state_interface name="position"/>
+                <state_interface name="velocity"/>
+            </joint>
+            <joint name="LoaderJoint">
+                <state_interface name="position"/>
+            </joint>
+            <joint name="HopperJoint">
+                <state_interface name="position"/>
+            </joint>
+            <joint name="DoorJoint">
+                <state_interface name="position"/>
+            </joint>
         </ros2_control>
     </xacro:unless>
@@ -52,4 +69,21 @@
                 <state_interface name="position"/>
             </joint>
+            <joint name="DW_Joint">
+                <state_interface name="position"/>
+                <state_interface name="velocity"/>
+            </joint>
+            <joint name="PW_Joint">
+                <state_interface name="position"/>
+                <state_interface name="velocity"/>
+            </joint>
+            <joint name="LoaderJoint">
+                <state_interface name="position"/>
+            </joint>
+            <joint name="HopperJoint">
+                <state_interface name="position"/>
+            </joint>
+            <joint name="DoorJoint">
+                <state_interface name="position"/>
+            </joint>
         </ros2_control>
     </xacro:if>

File: src/description/terrence.urdf.xacro (robot description, xacro)
@@ -4,9 +4,9 @@
   <xacro:arg name="sim_mode" default="false"/>
   <xacro:if value="$(arg use_ros2_control)">
-        <xacro:include filename="ros2_control.xacro"/>
-    </xacro:if>
-    <xacro:unless value="$(arg use_ros2_control)">
-        <xacro:include filename="gazebo_control.xacro"/>
-    </xacro:unless>
+      <xacro:include filename="ros2_control.xacro"/>
+  </xacro:if>
+  <xacro:unless value="$(arg use_ros2_control)">
+      <xacro:include filename="gazebo_control.xacro"/>
+  </xacro:unless>
   <link name="base_link" />
   <link name="base_footprint" />
@@ -18,6 +18,6 @@
   <link name="Base">
     <inertial>
-      <origin xyz="0.0071933 0.035942 -0.17341" rpy="0 0 0" />
-      <mass value="1.0994" />
+      <origin xyz="0.0071933 0.035942 -0.37341" rpy="0 0 0" />
+      <mass value="2.0994" />
       <inertia ixx="0.0052099" ixy="-7.8944E-22" ixz="-4.9264E-20" iyy="0.0060071" iyz="3.293E-21"
         izz="0.0014684" />
@@ -110,5 +110,5 @@
     <child link="DriverSprocket" />
     <axis xyz="1 0 0" />
-    <limit effort="10" velocity="0" />
+    <limit effort="10" velocity="10" />
   </joint>
   <gazebo reference="DriverSprocket">
@@ -178,5 +178,5 @@
     <child link="PassSprocket" />
     <axis xyz="1 0 0" />
-    <limit effort="10" velocity="0" />
+    <limit effort="10" velocity="10" />
   </joint>
   <gazebo reference="PassSprocket">
@@ -215,4 +215,6 @@
   <gazebo reference="Loader">
     <material>Gazebo/Red</material>
+    <mu1 value="0.001"/>
+    <mu2 value="0.001"/>
   </gazebo>
   <link name="Hopper">
