Commit message: Add required ros2_control files

File: src/description/ros2_control.xacro (robot description, xacro)
@@ -5,6 +5,6 @@
             <hardware>
                 <plugin>diffdrive_arduino/DiffDriveArduino</plugin>
-                <param name="left_wheel_name">left_wheel_joint</param>
-                <param name="right_wheel_name">right_wheel_joint</param>
+                <param name="DS_Joint">DS_Joint</param>
+                <param name="PS_Joint">PS_Joint</param>
                 <param name="loop_rate">30</param>
                 <param name="device">/dev/ttyUSB0</param>
@@ -13,5 +13,5 @@
                 <param name="enc_counts_per_rev">3450</param>
             </hardware>
-            <joint name="left_wheel_joint">
+            <joint name="DS_Joint">
                 <command_interface name="velocity">
                     <param name="min">-10</param>
@@ -21,5 +21,5 @@
                 <state_interface name="position"/>
             </joint>
-            <joint name="right_wheel_joint">
+            <joint name="PS_Joint">
                 <command_interface name="velocity">
                     <param name="min">-10</param>
@@ -36,5 +36,5 @@
                 <plugin>gz_ros2_control/GazeboSimSystem</plugin>
             </hardware>
-            <joint name="left_wheel_joint">
+            <joint name="DS_Joint">
                 <command_interface name="velocity">
                     <param name="min">-10</param>
@@ -44,5 +44,5 @@
                 <state_interface name="position"/>
             </joint>
-            <joint name="right_wheel_joint">
+            <joint name="PS_Joint">
                 <command_interface name="velocity">
                     <param name="min">-10</param>

File: src/description/terrence.urdf.xacro (robot description, xacro)
@@ -1,6 +1,12 @@
 <?xml version="1.0" encoding="utf-8"?>
 <robot xmlns:xacro="http://www.ros.org/wiki/xacro" name="LilT_Combined_URDF">
-  <xacro:arg name="sim_mode" default="false" />
-  <xacro:include filename="ros2_control.xacro" />
+  <xacro:arg name="use_ros2_control" default="true"/>
+  <xacro:arg name="sim_mode" default="false"/>
+  <xacro:if value="$(arg use_ros2_control)">
+        <xacro:include filename="ros2_control.xacro"/>
+    </xacro:if>
+    <xacro:unless value="$(arg use_ros2_control)">
+        <xacro:include filename="gazebo_control.xacro"/>
+    </xacro:unless>
   <link name="base_link" />
   <link name="base_footprint" />
@@ -38,4 +44,7 @@
     <child link="Base" />
   </joint>
+  <gazebo reference="Base">
+    <material>Gazebo/White</material>
+  </gazebo>
   <link name="DriverWheel">
     <inertial>
@@ -68,4 +77,9 @@
     <limit effort="10" velocity="0" />
   </joint>
+  <gazebo reference="DriverWheel">
+    <material>Gazebo/Blue</material>
+      <mu1 value="0.001"/>
+      <mu2 value="0.001"/>
+  </gazebo>
   <link name="DriverSprocket">
     <inertial>
@@ -98,4 +112,7 @@
     <limit effort="10" velocity="0" />
   </joint>
+  <gazebo reference="DriverSprocket">
+    <material>Gazebo/Blue</material>
+  </gazebo>
   <link name="PassWheel">
     <inertial>
@@ -128,4 +145,9 @@
     <limit effort="10" velocity="0" />
   </joint>
+  <gazebo reference="PassWheel">
+    <material>Gazebo/Blue</material>
+      <mu1 value="0.001"/>
+      <mu2 value="0.001"/>
+  </gazebo>
   <link name="PassSprocket">
     <inertial>
@@ -158,4 +180,7 @@
     <limit effort="10" velocity="0" />
   </joint>
+  <gazebo reference="PassSprocket">
+    <material>Gazebo/Blue</material>
+  </gazebo>
   <link name="Loader">
     <inertial>
@@ -188,4 +213,7 @@
     <limit lower="0" upper="1.571" effort="10" velocity="0.7854" />
   </joint>
+  <gazebo reference="Loader">
+    <material>Gazebo/Red</material>
+  </gazebo>
   <link name="Hopper">
     <inertial>
@@ -218,4 +246,7 @@
     <limit lower="0" upper="0.785" effort="10" velocity="0.3927" />
   </joint>
+  <gazebo reference="Hopper">
+    <material>Gazebo/White</material>
+  </gazebo>
   <link name="Door">
     <inertial>
@@ -248,3 +279,6 @@
     <limit lower="0" upper="0.3927" effort="0" velocity="0" />
   </joint>
+  <gazebo reference="Door">
+    <material>Gazebo/White</material>
+  </gazebo>
 </robot>

Commit message: fixed the hardware plugin name mismatch

File: src/description/ros2_control.xacro (robot description, xacro)
@@ -4,7 +4,6 @@
         <ros2_control name="RealRobot" type="system">
             <hardware>
-                <plugin>diffdrive_arduino/DiffDriveArduino</plugin>
-                <param name="DS_Joint">DS_Joint</param>
-                <param name="PS_Joint">PS_Joint</param>
+                <param name="left_wheel_name">DS_Joint</param>
+                <param name="right_wheel_name">PS_Joint</param>
                 <param name="loop_rate">30</param>
                 <param name="device">/dev/ttyUSB0</param>
@@ -12,41 +11,19 @@
                 <param name="timeout">1000</param>
             </hardware>
-            <joint name="DS_Joint">
+            <joint name="left_wheel_joint">
                 <command_interface name="velocity">
                     <param name="min">-10</param>
                     <param name="max">10</param>
                 </command_interface>
+                <state_interface name="position"/>
                 <state_interface name="velocity"/>
-                <state_interface name="position"/>
             </joint>
-            <joint name="PS_Joint">
+            <joint name="right_wheel_joint">
                 <command_interface name="velocity">
                     <param name="min">-10</param>
                     <param name="max">10</param>
                 </command_interface>
-                <state_interface name="velocity"/>
-                <state_interface name="position"/>
-            </joint>
-            <joint name="DW_Joint">
                 <state_interface name="position"/>
                 <state_interface name="velocity"/>
-            </joint>
-            <joint name="PW_Joint">
-                <state_interface name="position"/>
-                <state_interface name="velocity"/>
-            </joint>
-            <joint name="LoaderJoint">
-                <command_interface name="position">
-                    <param name="min">-1.57</param>  <!-- ~ -90 deg -->
-                    <param name="max"> 1.57</param>  <!-- ~  90 deg -->
-                </command_interface>
-                <state_interface name="position"/>
-                <state_interface name="velocity"/>
-            </joint>
-            <joint name="HopperJoint">
-                <state_interface name="position"/>
-            </joint>
-            <joint name="DoorJoint">
-                <state_interface name="position"/>
             </joint>
         </ros2_control>

Commit message: fixed name mismatches and working on fixing xacro joints for control

File: src/description/ros2_control.xacro (robot description, xacro)
@@ -10,21 +10,32 @@
                 <param name="device">/dev/ttyUSB0</param>
                 <param name="baud_rate">57600</param>
-                <param name="timeout">1000</param>
+                <param name="timeout_ms">1000</param>
+                <param name="enc_counts_per_rev">2944</param>
             </hardware>
-            <joint name="left_wheel_joint">
+            <joint name="DS_Joint">
                 <command_interface name="velocity">
-                    <param name="min">-10</param>
-                    <param name="max">10</param>
+                <param name="min">-10</param>
+                <param name="max">10</param>
+                </command_interface>
+                <state_interface name="velocity"/>
+                <state_interface name="position"/>
+            </joint>
+            <joint name="PS_Joint">
+                <command_interface name="velocity">
+                <param name="min">-10</param>
+                <param name="max">10</param>
+                </command_interface>
+                <state_interface name="velocity"/>
+                <state_interface name="position"/>
+            </joint>
+            <joint name="LoaderJoint">
+                <command_interface name="position">
+                <param name="min">-1.57</param>
+                <param name="max">1.57</param>
                 </command_interface>
                 <state_interface name="position"/>
-                <state_interface name="velocity"/>
             </joint>
-            <joint name="right_wheel_joint">
-                <command_interface name="velocity">
-                    <param name="min">-10</param>
-                    <param name="max">10</param>
-                </command_interface>
+            <joint name="DoorJoint">
                 <state_interface name="position"/>
-                <state_interface name="velocity"/>
             </joint>
         </ros2_control>

Commit message: changed from usb0 to acm0

File: src/description/ros2_control.xacro (robot description, xacro)
@@ -8,6 +8,6 @@
                 <param name="right_wheel_name">PS_Joint</param>
                 <param name="loop_rate">30</param>
-                <param name="device">/dev/ttyUSB0</param>
-                <param name="baud_rate">57600</param>
+                <param name="device">/dev/ttyACM0</param>
+                <param name="baud_rate">38400</param>
                 <param name="timeout_ms">1000</param>
                 <param name="enc_counts_per_rev">2944</param>
@@ -18,6 +18,6 @@
                 <param name="max">10</param>
                 </command_interface>
+                <state_interface name="position"/>
                 <state_interface name="velocity"/>
-                <state_interface name="position"/>
             </joint>
             <joint name="PS_Joint">
@@ -26,8 +26,8 @@
                 <param name="max">10</param>
                 </command_interface>
+                <state_interface name="position"/>
                 <state_interface name="velocity"/>
-                <state_interface name="position"/>
             </joint>
-            <joint name="LoaderJoint">
+            <!-- <joint name="LoaderJoint">
                 <command_interface name="position">
                 <param name="min">-1.57</param>
@@ -35,8 +35,9 @@
                 </command_interface>
                 <state_interface name="position"/>
+                <state_interface name="velocity"/>
             </joint>
             <joint name="DoorJoint">
                 <state_interface name="position"/>
-            </joint>
+            </joint> -->
         </ros2_control>
     </xacro:unless>
