Commit message: finished depth camera simulation

File: src/luna_test/description/depth_camera.xacro (robot description, xacro)
@@ -17,5 +17,5 @@
     <parent link="camera_link" />
     <child link="camera_link_optical" />
-    <origin xyz="0 0 0" rpy="-${pi/2} 0 $-{pi/2}" />
+    <origin xyz="0 0 0" rpy="${-pi/2} 0 ${-pi/2}" />
   </joint>
   <link name="camera_link_optical"></link>
@@ -29,5 +29,5 @@
         <horizontal_fov>1.089</horizontal_fov>
         <image>
-          <format>R8G8B8</format>
+          <format>B8G8R8</format>
           <width>640</width>
           <height>480</height>
@@ -39,5 +39,7 @@
       </camera>
       <plugin name="camera_controller" filename="libgazebo_ros_camera.so">
-        <frameName>camera_link_optical</frameName>
+        <frame_name>camera_link_optical</frame_name>
+        <min_depth>0.1</min_depth>
+        <max_depth>100.0</max_depth>
       </plugin>
     </sensor>
