Commit message: added base footprint link to robot core

File: src/luna_test/description/robot_core.xacro (robot description, xacro)
@@ -19,6 +19,12 @@
     </material>
     <!-- Base Link -->
-    <link name="base_link">
-    </link>
+    <link name="base_link"></link>
+    <!-- Base Footprint Link -->
+    <joint name="base_footprint_joint" type="fixed">
+        <parent link="base_link" />
+        <child link="base_footprint" />
+        <origin xyz="0 0 0" rpy="0 0 0" />
+    </joint>
+    <link name="base_footprint"></link>
     <!-- Chassis Link -->
     <joint name="chassis_joint" type="fixed">

Commit message: Updated for SLAM Toolbox

File: src/luna_test/description/robot_core.xacro (robot description, xacro)
@@ -26,5 +26,6 @@
         <origin xyz="0 0 0" rpy="0 0 0" />
     </joint>
-    <link name="base_footprint"></link>
+    <link name="base_footprint">
+    </link>
     <!-- Chassis Link -->
     <joint name="chassis_joint" type="fixed">
